File: projects/SG002/SG002.sch (KiCad schematic (older format))
At the start: 27 parts, among them J1 Conn_01x04, J2 Conn_01x02, J3 Conn_01x06, U1 74HC595N, U2 74HC595N, U3 74HC595N, U4 74HC595N, U5 74HC595N, U6 SST39VF3201_3202, U7 74LS166N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

Commit message: SG002 board initially completed.
Parts:
- C1, C2, C3, C4, C5, C6, C7, C8, D1, R1, R2, R3, R4, R5: footprint (none) -> alf64_mods:0805
- J1: footprint (none) -> alf64_mods:PINHEAD1x4
- J2, JP1: footprint (none) -> alf64_mods:PINHEAD1x2
- J3: footprint (none) -> alf64_mods:PINHEAD1x6
- R6: value 3.3k -> 3,3k; footprint (none) -> alf64_mods:0805
- U1, U2, U3, U4, U5, U7, U8: footprint (none) -> alf64_mods:SO16
- U6: footprint (none) -> alf64_mods:DIP48
Connections:
- net D0: now also U8.10 (E); no longer U8.14 (H)
- net D1: now also U8.12 (G); no longer U8.11 (F)
- net D14: now also U7.11 (F); no longer U7.12 (G)
- net D15: now also U7.14 (H); no longer U7.10 (E)
- net D6: now also U7.10 (E); no longer U7.14 (H)
- net D7: now also U7.12 (G); no longer U7.11 (F)
- net D8: now also U8.11 (F); no longer U8.12 (G)
- net D9: now also U8.14 (H); no longer U8.10 (E)
- net DATA_OUT: now also J3.5 (Pin_5); no longer J3.6 (Pin_6)
- net DATA_OUT_CLK: now also J3.4 (Pin_4); no longer J3.5 (Pin_5)
- net DATA_OUT_SHLD: now also J3.6 (Pin_6); no longer J3.4 (Pin_4)
- net SST_CE: now also J3.3 (Pin_3); no longer J3.2 (Pin_2)
- net SST_OE: now also J3.2 (Pin_2); no longer J3.1 (Pin_1)
- net SST_WE: now also J3.1 (Pin_1); no longer J3.3 (Pin_3)
Changed lines of the file:
@@
 F 0 "U7" H 9750 1950 50  0000 C CNN
 F 1 "74LS166N" H 9750 1750 50  0000 C CNN
-F 2 "" H 9750 1700 50  0001 C CNN
+F 2 "alf64_mods:SO16" H 9750 1700 50  0001 C CNN
 F 3 "" H 9750 1700 50  0001 C CNN
 	1    9750 1700
@@
 F 0 "U8" H 9750 4000 50  0000 C CNN
 F 1 "74LS166N" H 9750 3800 50  0000 C CNN
-F 2 "" H 9750 3750 50  0001 C CNN
+F 2 "alf64_mods:SO16" H 9750 3750 50  0001 C CNN
 F 3 "" H 9750 3750 50  0001 C CNN
 	1    9750 3750
@@
 F 0 "U1" H 2900 1800 50  0000 C CNN
 F 1 "74HC595N" H 2750 600 50  0000 C CNN
-F 2 "" H 2750 1200 50  0001 C CNN
+F 2 "alf64_mods:SO16" H 2750 1200 50  0001 C CNN
 F 3 "" H 2750 1200 50  0001 C CNN
 	1    2750 1200
@@
 F 0 "U2" H 2900 3250 50  0000 C CNN
 F 1 "74HC595N" H 2750 2050 50  0000 C CNN
-F 2 "" H 2750 2650 50  0001 C CNN
+F 2 "alf64_mods:SO16" H 2750 2650 50  0001 C CNN
 F 3 "" H 2750 2650 50  0001 C CNN
 	1    2750 2650
@@
 F 0 "U3" H 2900 4700 50  0000 C CNN
 F 1 "74HC595N" H 2750 3500 50  0000 C CNN
-F 2 "" H 2750 4100 50  0001 C CNN
+F 2 "alf64_mods:SO16" H 2750 4100 50  0001 C CNN
 F 3 "" H 2750 4100 50  0001 C CNN
 	1    2750 4100
@@
 F 0 "U4" H 2900 6150 50  0000 C CNN
 F 1 "74HC595N" H 2750 4950 50  0000 C CNN
-F 2 "" H 2750 5550 50  0001 C CNN
+F 2 "alf64_mods:SO16" H 2750 5550 50  0001 C CNN
 F 3 "" H 2750 5550 50  0001 C CNN
 	1    2750 5550
@@
 F 0 "U5" H 2900 7600 50  0000 C CNN
 F 1 "74HC595N" H 2750 6400 50  0000 C CNN
-F 2 "" H 2750 7000 50  0001 C CNN
+F 2 "alf64_mods:SO16" H 2750 7000 50  0001 C CNN
 F 3 "" H 2750 7000 50  0001 C CNN
 	1    2750 7000
@@
 F 0 "C1" H 5775 5800 50  0000 L CNN
 F 1 "100n" H 5775 5600 50  0000 L CNN
-F 2 "" H 5788 5550 50  0001 C CNN
+F 2 "alf64_mods:0805" H 5788 5550 50  0001 C CNN
 F 3 "" H 5750 5700 50  0001 C CNN
 	1    5750 5700
@@
 F 0 "C2" H 6025 5800 50  0000 L CNN
 F 1 "100n" H 6025 5600 50  0000 L CNN
-F 2 "" H 6038 5550 50  0001 C CNN
+F 2 "alf64_mods:0805" H 6038 5550 50  0001 C CNN
 F 3 "" H 6000 5700 50  0001 C CNN
 	1    6000 5700
@@
 F 0 "C3" H 6275 5800 50  0000 L CNN
 F 1 "100n" H 6275 5600 50  0000 L CNN
-F 2 "" H 6288 5550 50  0001 C CNN
+F 2 "alf64_mods:0805" H 6288 5550 50  0001 C CNN
 F 3 "" H 6250 5700 50  0001 C CNN
 	1    6250 5700
@@
 F 0 "C4" H 6525 5800 50  0000 L CNN
 F 1 "100n" H 6525 5600 50  0000 L CNN
-F 2 "" H 6538 5550 50  0001 C CNN
+F 2 "alf64_mods:0805" H 6538 5550 50  0001 C CNN
 F 3 "" H 6500 5700 50  0001 C CNN
 	1    6500 5700
@@
 F 0 "C5" H 6825 5800 50  0000 L CNN
 F 1 "100n" H 6825 5600 50  0000 L CNN
-F 2 "" H 6838 5550 50  0001 C CNN
+F 2 "alf64_mods:0805" H 6838 5550 50  0001 C CNN
 F 3 "" H 6800 5700 50  0001 C CNN
 	1    6800 5700
@@
 F 0 "C6" H 7075 5800 50  0000 L CNN
 F 1 "100n" H 7075 5600 50  0000 L CNN
-F 2 "" H 7088 5550 50  0001 C CNN
+F 2 "alf64_mods:0805" H 7088 5550 50  0001 C CNN
 F 3 "" H 7050 5700 50  0001 C CNN
 	1    7050 5700
@@
 F 0 "C7" H 7325 5800 50  0000 L CNN
 F 1 "100n" H 7325 5600 50  0000 L CNN
-F 2 "" H 7338 5550 50  0001 C CNN
+F 2 "alf64_mods:0805" H 7338 5550 50  0001 C CNN
 F 3 "" H 7300 5700 50  0001 C CNN
 	1    7300 5700
@@
 F 0 "C8" H 7575 5800 50  0000 L CNN
 F 1 "100n" H 7575 5600 50  0000 L CNN
-F 2 "" H 7588 5550 50  0001 C CNN
+F 2 "alf64_mods:0805" H 7588 5550 50  0001 C CNN
 F 3 "" H 7550 5700 50  0001 C CNN
 	1    7550 5700
@@
 F 0 "U6" H 6000 3200 60  0000 C CNN
 F 1 "SST39VF3201_3202" H 6000 700 60  0000 C CNN
-F 2 "" H 6000 1050 157 0001 C CNN
+F 2 "alf64_mods:DIP48" H 6000 1050 157 0001 C CNN
 F 3 "" H 6000 1050 157 0001 C CNN
 	1    6000 2100
@@
 F 0 "JP1" H 4950 3250 60  0000 C CNN
 F 1 "JMP" H 4950 3050 60  0000 C CNN
-F 2 "" H 4900 3150 60  0001 C CNN
+F 2 "alf64_mods:PINHEAD1x2" H 4900 3150 60  0001 C CNN
 F 3 "" H 4900 3150 60  0001 C CNN
 	1    4850 3150
@@
 F 0 "R2" V 6900 2700 50  0000 C CNN
 F 1 "10k" V 6950 2900 50  0000 C CNN
-F 2 "" V 6880 2900 50  0001 C CNN
+F 2 "alf64_mods:0805" V 6880 2900 50  0001 C CNN
 F 3 "" H 6950 2900 50  0001 C CNN
 	1    6950 2900
@@
 F 0 "R3" V 6900 2900 50  0000 C CNN
 F 1 "10k" V 6950 3100 50  0000 C CNN
-F 2 "" V 6880 3100 50  0001 C CNN
+F 2 "alf64_mods:0805" V 6880 3100 50  0001 C CNN
 F 3 "" H 6950 3100 50  0001 C CNN
 	1    6950 3100
@@
 F 0 "J2" H 5200 5750 50  0000 C CNN
 F 1 "Conn_01x02" H 5200 5450 50  0000 C CNN
-F 2 "" H 5200 5650 50  0001 C CNN
+F 2 "alf64_mods:PINHEAD1x2" H 5200 5650 50  0001 C CNN
 F 3 "" H 5200 5650 50  0001 C CNN
 	1    5200 5650
@@
 F 0 "J1" H 600 4350 50  0000 C CNN
 F 1 "Conn_01x04" H 450 3850 50  0000 C CNN
-F 2 "" H 600 4150 50  0001 C CNN
+F 2 "alf64_mods:PINHEAD1x4" H 600 4150 50  0001 C CNN
 F 3 "" H 600 4150 50  0001 C CNN
 	1    600  4150
@@
 F 0 "J3" H 5800 7250 50  0000 C CNN
 F 1 "Conn_01x06" H 5650 6550 50  0000 C CNN
-F 2 "" H 5800 6950 50  0001 C CNN
+F 2 "alf64_mods:PINHEAD1x6" H 5800 6950 50  0001 C CNN
 F 3 "" H 5800 6950 50  0001 C CNN
 	1    5800 6950
@@
 Wire Wire Line
 	4600 7250 5600 7250
+Text Label 4700 6850 0    60   ~ 0
+SST_OE
+Text Label 4700 6950 0    60   ~ 0
+SST_CE
 Text Label 4700 6750 0    60   ~ 0
-SST_OE
-Text Label 4700 6850 0    60   ~ 0
-SST_CE
-Text Label 4700 6950 0    60   ~ 0
 SST_WE
+Text Label 4700 7250 0    60   ~ 0
+DATA_OUT_SHLD
 Text Label 4700 7050 0    60   ~ 0
-DATA_OUT_SHLD
+DATA_OUT_CLK
 Text Label 4700 7150 0    60   ~ 0
-DATA_OUT_CLK
-Text Label 4700 7250 0    60   ~ 0
 DATA_OUT
 $Comp
@@
 F 0 "R1" H 1700 1050 50  0000 C CNN
 F 1 "10k" H 1700 1150 50  0000 C CNN
-F 2 "" V 1430 1100 50  0001 C CNN
+F 2 "alf64_mods:0805" V 1430 1100 50  0001 C CNN
 F 3 "" H 1500 1100 50  0001 C CNN
 	1    1500 1100
@@
 F 0 "R5" V 1300 4500 50  0000 C CNN
 F 1 "10k" V 1400 4450 50  0000 C CNN
-F 2 "" V 1330 4450 50  0001 C CNN
+F 2 "alf64_mods:0805" V 1330 4450 50  0001 C CNN
 F 3 "" H 1400 4450 50  0001 C CNN
 	1    1400 4450
@@
 F 0 "R4" H 7250 3450 50  0000 C CNN
 F 1 "10k" H 7250 3550 50  0000 C CNN
-F 2 "" V 7080 3400 50  0001 C CNN
+F 2 "alf64_mods:0805" V 7080 3400 50  0001 C CNN
 F 3 "" H 7150 3400 50  0001 C CNN
 	1    7150 3400
@@
 F 0 "D1" V 8150 5550 50  0000 C CNN
 F 1 "LED" V 8050 5550 50  0000 C CNN
-F 2 "" H 8100 5700 50  0001 C CNN
+F 2 "alf64_mods:0805" H 8100 5700 50  0001 C CNN
 F 3 "" H 8100 5700 50  0001 C CNN
 	1    8100 5700
@@
 P 7850 5500
 F 0 "R6" V 7750 5500 50  0000 C CNN
-F 1 "3.3k" V 7850 5500 50  0000 C CNN
-F 2 "" V 7780 5500 50  0001 C CNN
+F 1 "3,3k" V 7850 5500 50  0000 C CNN
+F 2 "alf64_mods:0805" V 7780 5500 50  0001 C CNN
 F 3 "" H 7850 5500 50  0001 C CNN
 	1    7850 5500
@@
 Text Label 7750 1450 0    60   ~ 0
 D4
-Text Label 7750 1550 0    60   ~ 0
-D15
-Text Label 7750 1650 0    60   ~ 0
-D7
-Text Label 7750 1750 0    60   ~ 0
-D14
-Text Label 7750 1850 0    60   ~ 0
-D6
 Text Label 7750 3200 0    60   ~ 0
 D11
@@
 Text Label 7750 3500 0    60   ~ 0
 D2
+Text Label 7750 3900 0    60   ~ 0
+D9
+Text Label 7750 3800 0    60   ~ 0
+D1
+Text Label 7750 3700 0    60   ~ 0
+D8
 Text Label 7750 3600 0    60   ~ 0
-D9
-Text Label 7750 3700 0    60   ~ 0
-D1
-Text Label 7750 3800 0    60   ~ 0
-D8
-Text Label 7750 3900 0    60   ~ 0
 D0
+Text Label 7750 1850 0    60   ~ 0
+D15
+Text Label 7750 1750 0    60   ~ 0
+D7
+Text Label 7750 1650 0    60   ~ 0
+D14
+Text Label 7750 1550 0    60   ~ 0
+D6
 $EndSCHEMATC
