File: projects/SG001/SG001.sch (KiCad schematic (older format))
At the start: 14 parts, among them U1 74LVC245, U2 74LVC245, U3 74LVC245, U4 SST39VF3201_3202, U5 LD1117S33TR

Commit message: SG001 initially completed.
Parts:
- C1: footprint (none) -> alf64_mods:2312
- C2, C3, C4, C5, C6: footprint (none) -> alf64_mods:0805
- CONN1, CONN2: footprint (none) -> alf64_mods:SG_cartconn
- JP1: footprint (none) -> alf64_mods:JMP1_SMD
- U1, U2, U3: footprint 74LVC245_SO20 -> alf64_mods:TSSOP20
- U4: footprint (none) -> alf64_mods:TSOP48_SST
- U5: footprint (none) -> alf64_mods:SOT223
Connections:
- net A21_5V: now also CONN2.9 (A21)
- no-connect marks 22 -> 21
Changed lines of the file:
@@
 F 0 "CONN1" H 2500 2800 60  0000 C CNN
 F 1 "SG_cartconn_sideA" H 2500 1000 60  0000 C CNN
-F 2 "" H 2500 1750 60  0001 C CNN
+F 2 "alf64_mods:SG_cartconn" H 2500 1750 60  0001 C CNN
 F 3 "" H 2500 1750 60  0001 C CNN
 	1    2500 2000
@@
 F 0 "CONN2" H 2550 5350 60  0000 C CNN
 F 1 "SG_cartconn_sideB" H 2550 3550 60  0000 C CNN
-F 2 "" H 2550 4200 60  0001 C CNN
+F 2 "alf64_mods:SG_cartconn" H 2550 4200 60  0001 C CNN
 F 3 "" H 2550 4200 60  0001 C CNN
 	1    2550 4500
@@
 $EndComp
 $Comp
-L GND_ #PWR2
+L GND_ #PWR01
 U 1 1 60908946
 P 1900 3050
-F 0 "#PWR2" H 1900 2800 50  0001 C CNN
+F 0 "#PWR01" H 1900 2800 50  0001 C CNN
 F 1 "GND_" H 1900 2900 50  0000 C CNN
 F 2 "" H 1900 3050 50  0001 C CNN
@@
 $EndComp
 $Comp
-L VCC_ #PWR1
+L VCC_ #PWR02
 U 1 1 609089CC
 P 1900 1000
-F 0 "#PWR1" H 1900 950 50  0001 C CNN
+F 0 "#PWR02" H 1900 950 50  0001 C CNN
 F 1 "VCC_" H 1900 1150 50  0000 C CNN
 F 2 "" H 1900 1000 50  0001 C CNN
@@
 F 0 "U1" H 5300 2250 60  0000 C CNN
 F 1 "74LVC245" H 5300 1050 60  0000 C CNN
-F 2 "74LVC245_SO20" H 5300 950 60  0001 C CNN
+F 2 "alf64_mods:TSSOP20" H 5300 950 60  0001 C CNN
 F 3 "" H 5300 1650 60  0001 C CNN
 	1    5300 1650
@@
 F 0 "U2" H 5300 3750 60  0000 C CNN
 F 1 "74LVC245" H 5300 2550 60  0000 C CNN
-F 2 "74LVC245_SO20" H 5300 2450 60  0001 C CNN
+F 2 "alf64_mods:TSSOP20" H 5300 2450 60  0001 C CNN
 F 3 "" H 5300 3150 60  0001 C CNN
 	1    5300 3150
@@
 F 0 "U3" H 5300 5300 60  0000 C CNN
 F 1 "74LVC245" H 5300 4100 60  0000 C CNN
-F 2 "74LVC245_SO20" H 5300 4000 60  0001 C CNN
+F 2 "alf64_mods:TSSOP20" H 5300 4000 60  0001 C CNN
 F 3 "" H 5300 4700 60  0001 C CNN
 	1    5300 4700
@@
 $EndComp
 $Comp
-L GND_ #PWR5
+L GND_ #PWR03
 U 1 1 6090AC40
 P 4650 5350
-F 0 "#PWR5" H 4650 5100 50  0001 C CNN
+F 0 "#PWR03" H 4650 5100 50  0001 C CNN
 F 1 "GND_" H 4650 5200 50  0000 C CNN
 F 2 "" H 4650 5350 50  0001 C CNN
@@
 $EndComp
 $Comp
-L +3V3_ #PWR4
+L +3V3_ #PWR04
 U 1 1 6090AFC5
 P 4550 900
-F 0 "#PWR4" H 4550 850 50  0001 C CNN
+F 0 "#PWR04" H 4550 850 50  0001 C CNN
 F 1 "+3V3_" H 4550 1040 50  0000 C CNN
 F 2 "" H 4550 900 50  0001 C CNN
@@
 $EndComp
 $Comp
-L GND_ #PWR6
+L GND_ #PWR05
 U 1 1 6090B14B
 P 6000 5350
-F 0 "#PWR6" H 6000 5100 50  0001 C CNN
+F 0 "#PWR05" H 6000 5100 50  0001 C CNN
 F 1 "GND_" H 6000 5200 50  0000 C CNN
 F 2 "" H 6000 5350 50  0001 C CNN
@@
 $EndComp
 $Comp
-L +3V3_ #PWR7
+L +3V3_ #PWR06
 U 1 1 6090B473
 P 6100 900
-F 0 "#PWR7" H 6100 850 50  0001 C CNN
+F 0 "#PWR06" H 6100 850 50  0001 C CNN
 F 1 "+3V3_" H 6100 1040 50  0000 C CNN
 F 2 "" H 6100 900 50  0001 C CNN
@@
 $EndComp
 $Comp
-L +3V3_ #PWR11
+L +3V3_ #PWR07
 U 1 1 6090B640
 P 9000 950
-F 0 "#PWR11" H 9000 900 50  0001 C CNN
+F 0 "#PWR07" H 9000 900 50  0001 C CNN
 F 1 "+3V3_" H 9000 1090 50  0000 C CNN
 F 2 "" H 9000 950 50  0001 C CNN
@@
 NoConn ~ 3150 4950
 NoConn ~ 3150 4850
-NoConn ~ 3150 4250
 NoConn ~ 3150 4350
 NoConn ~ 3150 4450
@@
 	6850 3300 6950 3200
 $Comp
-L GND_ #PWR12
+L GND_ #PWR08
 U 1 1 6090E06A
 P 9000 3650
-F 0 "#PWR12" H 9000 3400 50  0001 C CNN
+F 0 "#PWR08" H 9000 3400 50  0001 C CNN
 F 1 "GND_" H 9000 3500 50  0000 C CNN
 F 2 "" H 9000 3650 50  0001 C CNN
@@
 $EndComp
 $Comp
-L +3V3_ #PWR8
+L +3V3_ #PWR09
 U 1 1 6090E64F
 P 7700 950
-F 0 "#PWR8" H 7700 900 50  0001 C CNN
+F 0 "#PWR09" H 7700 900 50  0001 C CNN
 F 1 "+3V3_" H 7700 1090 50  0000 C CNN
 F 2 "" H 7700 950 50  0001 C CNN
@@
 DQ15_3V
 $Comp
-L GND_ #PWR3
+L GND_ #PWR010
 U 1 1 60910973
 P 3150 5350
-F 0 "#PWR3" H 3150 5100 50  0001 C CNN
+F 0 "#PWR010" H 3150 5100 50  0001 C CNN
 F 1 "GND_" H 3150 5200 50  0000 C CNN
 F 2 "" H 3150 5350 50  0001 C CNN
@@
 F 0 "U5" H 8300 4850 50  0000 C CNN
 F 1 "LD1117S33TR" H 8450 4850 50  0000 L CNN
-F 2 "" H 7650 4850 50  0001 C CNN
+F 2 "alf64_mods:SOT223" H 7650 4850 50  0001 C CNN
 F 3 "" H 7750 4450 50  0001 C CNN
 	1    8500 4650
@@
 $EndComp
 $Comp
-L VCC_ #PWR9
+L VCC_ #PWR011
 U 1 1 60908233
 P 8000 4400
-F 0 "#PWR9" H 8000 4350 50  0001 C CNN
+F 0 "#PWR011" H 8000 4350 50  0001 C CNN
 F 1 "VCC_" H 8000 4550 50  0000 C CNN
 F 2 "" H 8000 4400 50  0001 C CNN
@@
 $EndComp
 $Comp
-L +3V3_ #PWR13
+L +3V3_ #PWR012
 U 1 1 609082D1
 P 9300 4400
-F 0 "#PWR13" H 9300 4350 50  0001 C CNN
+F 0 "#PWR012" H 9300 4350 50  0001 C CNN
 F 1 "+3V3_" H 9300 4540 50  0000 C CNN
 F 2 "" H 9300 4400 50  0001 C CNN
@@
 NoConn ~ 8550 5050
 $Comp
-L GND_ #PWR10
+L GND_ #PWR013
 U 1 1 60908619
 P 8450 5350
-F 0 "#PWR10" H 8450 5100 50  0001 C CNN
+F 0 "#PWR013" H 8450 5100 50  0001 C CNN
 F 1 "GND_" H 8450 5200 50  0000 C CNN
 F 2 "" H 8450 5350 50  0001 C CNN
@@
 $EndComp
 $Comp
-L PWR_FLAG #FLG1
+L PWR_FLAG #FLG014
 U 1 1 60908A9B
 P 7550 4500
-F 0 "#FLG1" H 7550 4575 50  0001 C CNN
+F 0 "#FLG014" H 7550 4575 50  0001 C CNN
 F 1 "PWR_FLAG" H 7550 4650 50  0000 C CNN
 F 2 "" H 7550 4500 50  0001 C CNN
@@
 $EndComp
 $Comp
-L PWR_FLAG #FLG2
+L PWR_FLAG #FLG015
 U 1 1 60908AC4
 P 7550 5350
-F 0 "#FLG2" H 7550 5425 50  0001 C CNN
+F 0 "#FLG015" H 7550 5425 50  0001 C CNN
 F 1 "PWR_FLAG" H 7550 5500 50  0000 C CNN
 F 2 "" H 7550 5350 50  0001 C CNN
@@
 $EndComp
 $Comp
-L PWR_FLAG #FLG3
+L PWR_FLAG #FLG016
 U 1 1 60909128
 P 9800 4400
-F 0 "#FLG3" H 9800 4475 50  0001 C CNN
+F 0 "#FLG016" H 9800 4475 50  0001 C CNN
 F 1 "PWR_FLAG" H 9800 4550 50  0000 C CNN
 F 2 "" H 9800 4400 50  0001 C CNN
@@
 F 0 "C3" H 9075 5200 50  0000 L CNN
 F 1 "100n" H 9075 5000 50  0000 L CNN
-F 2 "" H 9088 4950 50  0001 C CNN
+F 2 "alf64_mods:0805" H 9088 4950 50  0001 C CNN
 F 3 "" H 9050 5100 50  0001 C CNN
 	1    9050 5100
@@
 F 0 "C4" H 9325 5200 50  0000 L CNN
 F 1 "100n" H 9325 5000 50  0000 L CNN
-F 2 "" H 9338 4950 50  0001 C CNN
+F 2 "alf64_mods:0805" H 9338 4950 50  0001 C CNN
 F 3 "" H 9300 5100 50  0001 C CNN
 	1    9300 5100
@@
 F 0 "C5" H 9575 5200 50  0000 L CNN
 F 1 "100n" H 9575 5000 50  0000 L CNN
-F 2 "" H 9588 4950 50  0001 C CNN
+F 2 "alf64_mods:0805" H 9588 4950 50  0001 C CNN
 F 3 "" H 9550 5100 50  0001 C CNN
 	1    9550 5100
@@
 F 0 "C6" H 9825 5200 50  0000 L CNN
 F 1 "100n" H 9825 5000 50  0000 L CNN
-F 2 "" H 9838 4950 50  0001 C CNN
+F 2 "alf64_mods:0805" H 9838 4950 50  0001 C CNN
 F 3 "" H 9800 5100 50  0001 C CNN
 	1    9800 5100
@@
 F 0 "C2" H 8025 5200 50  0000 L CNN
 F 1 "100n" H 8025 5000 50  0000 L CNN
-F 2 "" H 8038 4950 50  0001 C CNN
+F 2 "alf64_mods:0805" H 8038 4950 50  0001 C CNN
 F 3 "" H 8000 5100 50  0001 C CNN
 	1    8000 5100
@@
 F 0 "C1" H 7725 5200 50  0000 L CNN
 F 1 "47u 16V" H 7350 5000 50  0000 L CNN
-F 2 "" H 7738 4950 50  0001 C CNN
+F 2 "alf64_mods:2312" H 7738 4950 50  0001 C CNN
 F 3 "" H 7700 5100 50  0001 C CNN
 	1    7700 5100
@@
 F 0 "U4" H 8350 3400 60  0000 C CNN
 F 1 "SST39VF3201_3202" H 8350 900 60  0000 C CNN
-F 2 "" H 8350 1250 157 0001 C CNN
+F 2 "alf64_mods:TSOP48_SST" H 8350 1250 157 0001 C CNN
 F 3 "" H 8350 1250 157 0001 C CNN
 	1    8350 2300
@@
 F 0 "JP1" H 7400 3500 60  0000 C CNN
 F 1 "JMP" H 7400 3300 60  0000 C CNN
-F 2 "" H 7450 3400 60  0001 C CNN
+F 2 "alf64_mods:JMP1_SMD" H 7450 3400 60  0001 C CNN
 F 3 "" H 7450 3400 60  0001 C CNN
 	1    7400 3400
@@
 Wire Wire Line
 	4000 3000 4750 3000
-Wire Wire Line
-	4000 3100 4750 3100
 Wire Wire Line
 	4000 3200 4750 3200
@@
 	2000 4150 1900 4150
 Wire Wire Line
-	3050 4250 3150 4250
+	3050 4250 3800 4250
 Wire Wire Line
 	3050 4350 3150 4350
@@
 Text Label 4100 1300 0    60   ~ 0
 A17_5V
+Wire Wire Line
+	4000 3100 4750 3100
+Entry Wire Line
+	3800 4250 3900 4350
+Text Label 3250 4250 0    60   ~ 0
+A21_5V
 $EndSCHEMATC
