File: projects/SG001/SG001.kicad_pcb (KiCad board)
At the start: 2 copper layers, 83.6 x 40 mm, 16 parts, among them M6_1 HOLE_M6, M6_2 HOLE_M6, U1 74LVC245, U2 74LVC245, U3 74LVC245, U4 SST39VF3201_3202, U5 LD1117S33TR

Commit message: SG001 completed.
Routing:
- net GND_: track 262.3 -> 549.5 mm, vias 9 -> 89
- net +3V3_: track 93.6 -> 110.2 mm, vias 4 -> 3
- net /A06_5V: track 34.0 -> 31.7 mm
- net VCC_: track 124.0 -> 125.6 mm
Other:
- rule pad_to_mask_clearance: 0.2 -> 0.1
- board text added: "001P1"
- board text added: "A1"
- board text added: "A16"
- board text added: "A24"
- board text added: "A32"
- board text added: "A8"
- board text added: "B1"
- board text added: "B15"
- board text added: "B21"
- board text added: "B31"
- board text added: "SG"

Commit message: SG001 fixes, gerbers generated and board released as SG001P1.
Routing:
- net GND_: track 549.5 -> 550.6 mm

Commit message: SG001 40mm dimension increased to 45mm, because of manufacturer request (board needs to be at least 45mm wide for bevelling to be possible to apply) SG001 gerbers re-generated and board released as SG001P2.
Routing:
- net GND_: track 550.6 -> 608.8 mm, vias 89 -> 100
Other:
- board size 83.6 x 40 mm -> 83.6 x 45 mm
- board text added: "001P2"
- board text removed: "001P1"
